Commit message: Bno055 entegre edildi

File: pilbot_description/urdf/pilbot.urdf.xacro (robot description, xacro)
@@ -145,4 +145,31 @@
         <axis xyz="0 0 0" />
     </joint>
+    <link name="imu_link">
+        <inertial>
+            <origin xyz="-0.00552433659106688 0.000168210391520346 0.000514000497342681" rpy="0 0 0" />
+            <mass value="0.000528415362211671" />
+            <inertia ixx="1.46176048428261E-08" ixy="1.40015117949421E-10" ixz="-1.99633872937403E-12"
+                    iyy="8.59662482954888E-09" iyz="7.52375112767959E-12"
+                    izz="2.30279421279312E-08" />
+        </inertial>
+        <visual>
+            <origin xyz="0 0 0" rpy="0 0 0"/>
+            <geometry>
+                <mesh filename="package://pilbot_description/meshes/imu_link.STL"/>
+            </geometry>
+            <material name="silver" />
+        </visual>
+        <collision>
+            <origin xyz="0 0 0" rpy="0 0 0"/>
+            <geometry>
+               <mesh filename="package://pilbot_description/meshes/imu_link.STL"/>
+            </geometry>
+        </collision>
+    </link>
+    <joint name="imu_joint" type="fixed">
+        <origin xyz="0 0 0.07" rpy="3.14 0 0"/>
+        <parent link="base_link"/>
+        <child link="imu_link"/>
+    </joint>
     <material name="blue">
         <color rgba="0 0 1 1"/>

File: pilbot_description/urdf/pilbot_gazebo.xacro (robot description, xacro)
@@ -40,4 +40,58 @@
             <parameters>$(find pilbot_controller)/config/controller.yaml</parameters>
         </plugin>
+        <plugin filename="ignition-gazebo-imu-system" name="ignition::gazebo::systems::Imu"></plugin>
+    </gazebo>
+    <!-- bno055 -->
+    <!-- Based on bno055 datasheet-->
+    <!-- https://www.bosch-sensortec.com/media/boschsensortec/downloads/datasheets/bst-bno055-ds000.pdf -->
+    <gazebo reference="imu_link">
+        <sensor name="imu" type="imu">
+            <always_on>true</always_on>
+            <update_rate>100</update_rate>
+            <gz_frame_id>imu_link</gz_frame_id>
+            <topic>imu</topic>
+            <imu>
+                <angular_velocity>
+                    <x>
+                        <noise type="gaussian">
+                            <mean>0.0</mean>
+                            <stddev>0.00174532925</stddev> <!-- variance -->
+                        </noise>
+                    </x>
+                    <y>
+                        <noise type="gaussian">
+                            <mean>0.0</mean>
+                            <stddev>0.00174532925</stddev>
+                        </noise>
+                    </y>
+                    <z>
+                        <noise type="gaussian">
+                            <mean>0.0</mean>
+                            <stddev>0.00174532925</stddev>
+                        </noise>
+                    </z>
+                </angular_velocity>
+                <linear_acceleration>
+                    <x>
+                        <noise type="gaussian">
+                            <mean>0.0</mean>
+                            <stddev>0.0014715</stddev> <!-- variance, noise -->
+                        </noise>
+                    </x>
+                    <y>
+                        <noise type="gaussian">
+                            <mean>0.0</mean>
+                            <stddev>0.0014715</stddev> <!-- variance -->
+                        </noise>
+                    </y>
+                    <z>
+                        <noise type="gaussian">
+                            <mean>0.0</mean>
+                            <stddev>0.0014715</stddev> <!-- variance -->
+                        </noise>
+                    </z>
+                </linear_acceleration>
+            </imu>
+        </sensor>
     </gazebo>
 </robot>

Commit message: 3 tane imu eklendi ancak kod daha dinamik hale getirilmeli, ayrıca imu logger oluşturuldu

File: pilbot_description/urdf/pilbot.urdf.xacro (robot description, xacro)
@@ -145,5 +145,5 @@
         <axis xyz="0 0 0" />
     </joint>
-    <link name="imu_link">
+    <link name="imu_link1">
         <inertial>
             <origin xyz="-0.00552433659106688 0.000168210391520346 0.000514000497342681" rpy="0 0 0" />
@@ -167,8 +167,62 @@
         </collision>
     </link>
-    <joint name="imu_joint" type="fixed">
+    <joint name="imu_joint1" type="fixed">
         <origin xyz="0 0 0.07" rpy="3.14 0 0"/>
         <parent link="base_link"/>
-        <child link="imu_link"/>
+        <child link="imu_link1"/>
+    </joint>
+    <link name="imu_link2">
+        <inertial>
+            <origin xyz="-0.00552433659106688 0.000168210391520346 0.000514000497342681" rpy="0 0 0" />
+            <mass value="0.000528415362211671" />
+            <inertia ixx="1.46176048428261E-08" ixy="1.40015117949421E-10" ixz="-1.99633872937403E-12"
+                    iyy="8.59662482954888E-09" iyz="7.52375112767959E-12"
+                    izz="2.30279421279312E-08" />
+        </inertial>
+        <visual>
+            <origin xyz="0 0 0" rpy="0 0 0"/>
+            <geometry>
+                <mesh filename="package://pilbot_description/meshes/imu_link.STL"/>
+            </geometry>
+            <material name="silver" />
+        </visual>
+        <collision>
+            <origin xyz="0 0 0" rpy="0 0 0"/>
+            <geometry>
+               <mesh filename="package://pilbot_description/meshes/imu_link.STL"/>
+            </geometry>
+        </collision>
+    </link>
+    <joint name="imu_joint2" type="fixed">
+        <origin xyz="0 0 0.07" rpy="3.14 0 0"/>
+        <parent link="base_link"/>
+        <child link="imu_link2"/>
+    </joint>
+    <link name="imu_link3">
+        <inertial>
+            <origin xyz="-0.00552433659106688 0.000168210391520346 0.000514000497342681" rpy="0 0 0" />
+            <mass value="0.000528415362211671" />
+            <inertia ixx="1.46176048428261E-08" ixy="1.40015117949421E-10" ixz="-1.99633872937403E-12"
+                    iyy="8.59662482954888E-09" iyz="7.52375112767959E-12"
+                    izz="2.30279421279312E-08" />
+        </inertial>
+        <visual>
+            <origin xyz="0 0 0" rpy="0 0 0"/>
+            <geometry>
+                <mesh filename="package://pilbot_description/meshes/imu_link.STL"/>
+            </geometry>
+            <material name="silver" />
+        </visual>
+        <collision>
+            <origin xyz="0 0 0" rpy="0 0 0"/>
+            <geometry>
+               <mesh filename="package://pilbot_description/meshes/imu_link.STL"/>
+            </geometry>
+        </collision>
+    </link>
+    <joint name="imu_joint3" type="fixed">
+        <origin xyz="0 0 0.07" rpy="3.14 0 0"/>
+        <parent link="base_link"/>
+        <child link="imu_link3"/>
     </joint>
     <material name="blue">

File: pilbot_description/urdf/pilbot_gazebo.xacro (robot description, xacro)
@@ -45,10 +45,110 @@
     <!-- Based on bno055 datasheet-->
     <!-- https://www.bosch-sensortec.com/media/boschsensortec/downloads/datasheets/bst-bno055-ds000.pdf -->
-    <gazebo reference="imu_link">
-        <sensor name="imu" type="imu">
+    <gazebo reference="imu_link1">
+        <sensor name="imu1" type="imu">
             <always_on>true</always_on>
             <update_rate>100</update_rate>
-            <gz_frame_id>imu_link</gz_frame_id>
-            <topic>imu</topic>
+            <gz_frame_id>imu_link1</gz_frame_id>
+            <topic>imu1</topic>
+            <imu>
+                <angular_velocity>
+                    <x>
+                        <noise type="gaussian">
+                            <mean>0.0</mean>
+                            <stddev>0.00174532925</stddev> <!-- variance -->
+                        </noise>
+                    </x>
+                    <y>
+                        <noise type="gaussian">
+                            <mean>0.0</mean>
+                            <stddev>0.00174532925</stddev>
+                        </noise>
+                    </y>
+                    <z>
+                        <noise type="gaussian">
+                            <mean>0.0</mean>
+                            <stddev>0.00174532925</stddev>
+                        </noise>
+                    </z>
+                </angular_velocity>
+                <linear_acceleration>
+                    <x>
+                        <noise type="gaussian">
+                            <mean>0.0</mean>
+                            <stddev>0.0014715</stddev> <!-- variance, noise -->
+                        </noise>
+                    </x>
+                    <y>
+                        <noise type="gaussian">
+                            <mean>0.0</mean>
+                            <stddev>0.0014715</stddev> <!-- variance -->
+                        </noise>
+                    </y>
+                    <z>
+                        <noise type="gaussian">
+                            <mean>0.0</mean>
+                            <stddev>0.0014715</stddev> <!-- variance -->
+                        </noise>
+                    </z>
+                </linear_acceleration>
+            </imu>
+        </sensor>
+    </gazebo>
+    <gazebo reference="imu_link2">
+        <sensor name="imu2" type="imu">
+            <always_on>true</always_on>
+            <update_rate>100</update_rate>
+            <gz_frame_id>imu_link2</gz_frame_id>
+            <topic>imu2</topic>
+            <imu>
+                <angular_velocity>
+                    <x>
+                        <noise type="gaussian">
+                            <mean>0.0</mean>
+                            <stddev>0.00174532925</stddev> <!-- variance -->
+                        </noise>
+                    </x>
+                    <y>
+                        <noise type="gaussian">
+                            <mean>0.0</mean>
+                            <stddev>0.00174532925</stddev>
+                        </noise>
+                    </y>
+                    <z>
+                        <noise type="gaussian">
+                            <mean>0.0</mean>
+                            <stddev>0.00174532925</stddev>
+                        </noise>
+                    </z>
+                </angular_velocity>
+                <linear_acceleration>
+                    <x>
+                        <noise type="gaussian">
+                            <mean>0.0</mean>
+                            <stddev>0.0014715</stddev> <!-- variance, noise -->
+                        </noise>
+                    </x>
+                    <y>
+                        <noise type="gaussian">
+                            <mean>0.0</mean>
+                            <stddev>0.0014715</stddev> <!-- variance -->
+                        </noise>
+                    </y>
+                    <z>
+                        <noise type="gaussian">
+                            <mean>0.0</mean>
+                            <stddev>0.0014715</stddev> <!-- variance -->
+                        </noise>
+                    </z>
+                </linear_acceleration>
+            </imu>
+        </sensor>
+    </gazebo>
+    <gazebo reference="imu_link3">
+        <sensor name="imu3" type="imu">
+            <always_on>true</always_on>
+            <update_rate>100</update_rate>
+            <gz_frame_id>imu_link3</gz_frame_id>
+            <topic>imu3</topic>
             <imu>
                 <angular_velocity>

Commit message: Tf'ler ve ros2 control ayarlandı

File: pilbot_description/urdf/pilbot.urdf.xacro (robot description, xacro)
@@ -168,5 +168,5 @@
     </link>
     <joint name="imu_joint1" type="fixed">
-        <origin xyz="0 0 0.07" rpy="3.14 0 0"/>
+        <origin xyz="0 0 0.07" rpy="0 0 0"/>
         <parent link="base_link"/>
         <child link="imu_link1"/>
@@ -195,5 +195,5 @@
     </link>
     <joint name="imu_joint2" type="fixed">
-        <origin xyz="0 0 0.07" rpy="3.14 0 0"/>
+        <origin xyz="0 0 0.07" rpy="0 0 0"/>
         <parent link="base_link"/>
         <child link="imu_link2"/>
@@ -222,5 +222,5 @@
     </link>
     <joint name="imu_joint3" type="fixed">
-        <origin xyz="0 0 0.07" rpy="3.14 0 0"/>
+        <origin xyz="0 0 0.07" rpy="0 0 0"/>
         <parent link="base_link"/>
         <child link="imu_link3"/>

File: pilbot_description/urdf/pilbot_gazebo.xacro (robot description, xacro)
@@ -41,4 +41,7 @@
         </plugin>
         <plugin filename="ignition-gazebo-imu-system" name="ignition::gazebo::systems::Imu"></plugin>
+        <plugin filename="libignition-gazebo-sensors-system.so" name="ignition::gazebo::systems::Sensors">
+            <render_engine>ogre2</render_engine>
+        </plugin>
         <plugin filename="ignition-gazebo-odometry-publisher-system" name="ignition::gazebo::systems::OdometryPublisher">
             <robot_base_frame>base_footprint</robot_base_frame>
@@ -56,5 +59,5 @@
             <always_on>true</always_on>
             <update_rate>100</update_rate>
-            <gz_frame_id>imu_link1</gz_frame_id>
+            <gz_frame_id>imu1_link</gz_frame_id>
             <topic>imu1</topic>
             <imu>
@@ -63,17 +66,23 @@
                         <noise type="gaussian">
                             <mean>0.0</mean>
-                            <stddev>0.00174532925</stddev> <!-- variance -->
-                        </noise>
-                    </x>
-                    <y>
-                        <noise type="gaussian">
-                            <mean>0.0</mean>
-                            <stddev>0.00174532925</stddev>
-                        </noise>
-                    </y>
-                    <z>
-                        <noise type="gaussian">
-                            <mean>0.0</mean>
-                            <stddev>0.00174532925</stddev>
+                            <stddev>0.001745329251</stddev>  <!-- Noise Density, radyan cinsinden! (sensörün tipik davranışı modellenmiştir) -->
+                            <bias_mean>0.0</bias_mean>
+                            <bias_stddev>0.01745329251</bias_stddev> <!-- Bias instability, radyan cinsinden! (sensörün tipik davranışı modellenmiştir) -->
+                        </noise>
+                    </x>
+                    <y>
+                        <noise type="gaussian">
+                            <mean>0.0</mean>
+                            <stddev>0.001745329251</stddev>
+                            <bias_mean>0.0</bias_mean>
+                            <bias_stddev>0.01745329251</bias_stddev>
+                        </noise>
+                    </y>
+                    <z>
+                        <noise type="gaussian">
+                            <mean>0.0</mean>
+                            <stddev>0.001745329251</stddev>
+                            <bias_mean>0.0</bias_mean>
+                            <bias_stddev>0.01745329251</bias_stddev>
                         </noise>
                     </z>
@@ -82,19 +91,25 @@
                     <x>
                         <noise type="gaussian">
-                            <mean>0.0</mean>
-                            <stddev>0.0014715</stddev> <!-- variance, noise -->
-                        </noise>
-                    </x>
-                    <y>
-                        <noise type="gaussian">
-                            <mean>0.0</mean>
-                            <stddev>0.0014715</stddev> <!-- variance -->
-                        </noise>
-                    </y>
-                    <z>
-                        <noise type="gaussian">
-                            <mean>0.0</mean>
-                            <stddev>0.0014715</stddev> <!-- variance -->
-                        </noise>
+                            <mean>0.0</mean>    <!-- 100 ODR(Output Data Rate) için 32hz bandwith-->
+                            <stddev>8.32e-3</stddev> <!-- Output Noise Density, m/s^2 cinsinde, sensorün tipik davranışı ele alınmıştır. -->
+                            <bias_mean>0.0</bias_mean>
+                            <bias_stddev>0.4903</bias_stddev>
+                        </noise>
+                    </x>
+                    <y>
+                    <noise type="gaussian">
+                        <mean>0.0</mean>
+                        <stddev>1.8639e-5</stddev>
+                        <bias_mean>0.0</bias_mean>
+                        <bias_stddev>1.471e-3</bias_stddev>
+                    </noise>
+                    </y>
+                    <z>
+                    <noise type="gaussian">
+                        <mean>0.0</mean>
+                        <stddev>1.8639e-5</stddev>
+                        <bias_mean>0.0</bias_mean>
+                        <bias_stddev>1.471e-3</bias_stddev>
+                    </noise>
                     </z>
                 </linear_acceleration>
@@ -106,5 +121,5 @@
             <always_on>true</always_on>
             <update_rate>100</update_rate>
-            <gz_frame_id>imu_link2</gz_frame_id>
+            <gz_frame_id>imu2_link</gz_frame_id>
             <topic>imu2</topic>
             <imu>
@@ -156,5 +171,5 @@
             <always_on>true</always_on>
             <update_rate>100</update_rate>
-            <gz_frame_id>imu_link3</gz_frame_id>
+            <gz_frame_id>imu3_link</gz_frame_id>
             <topic>imu3</topic>
             <imu>
