Commit message: Test ortamı hazırlandı, çoğu hata düzeltildi

File: pilbot_description/urdf/pilbot.urdf.xacro (robot description, xacro)
@@ -112,5 +112,5 @@
     </link>
     <joint name="caster_front_joint" type="fixed">
-        <origin xyz="0.04755 0 -0.0275" rpy="0 0 0" />
+        <origin xyz="0.04755 0 -0.028" rpy="0 0 0" />
         <parent link="base_link" />
         <child link="caster_front_link" />
@@ -140,5 +140,5 @@
     </link>
     <joint name="caster_rear_joint" type="fixed">
-        <origin xyz="-0.04755 0 -0.0275" rpy="0 0 0" />
+        <origin xyz="-0.04755 0 -0.028" rpy="0 0 0" />
         <parent link="base_link" />
         <child link="caster_rear_link" />

File: pilbot_description/urdf/pilbot_gazebo.xacro (robot description, xacro)
@@ -64,23 +64,23 @@
                         <noise type="gaussian">
                             <mean>0.0</mean>
-                            <stddev>0.000006108</stddev>
-                            <bias_mean>0.0</bias_mean>
-                            <bias_stddev>0.00002424</bias_stddev>
-                        </noise>
-                    </x>
-                    <y>
-                        <noise type="gaussian">
-                            <mean>0.0</mean>
-                            <stddev>0.000006108</stddev>
-                            <bias_mean>0.0</bias_mean>
-                            <bias_stddev>0.00002424</bias_stddev>
-                        </noise>
-                    </y>
-                    <z>
-                        <noise type="gaussian">
-                            <mean>0.0</mean>
-                            <stddev>0.000006108</stddev>
-                            <bias_mean>0.0</bias_mean>
-                            <bias_stddev>0.00002424</bias_stddev>
+                            <stddev>0.0006109</stddev>
+                            <bias_mean>0.0</bias_mean>
+                            <bias_stddev>0.00004848</bias_stddev>
+                        </noise>
+                    </x>
+                    <y>
+                        <noise type="gaussian">
+                            <mean>0.0</mean>
+                            <stddev>0.0006109</stddev>
+                            <bias_mean>0.0</bias_mean>
+                            <bias_stddev>0.00004848</bias_stddev>
+                        </noise>
+                    </y>
+                    <z>
+                        <noise type="gaussian">
+                            <mean>0.0</mean>
+                            <stddev>0.0006109</stddev>
+                            <bias_mean>0.0</bias_mean>
+                            <bias_stddev>0.00004848</bias_stddev>
                         </noise>
                     </z>
@@ -90,5 +90,5 @@
                         <noise type="gaussian">
                             <mean>0.0</mean>
-                            <stddev>0.0001373</stddev>
+                            <stddev>0.01373</stddev>
                             <bias_mean>0.0</bias_mean>
                             <bias_stddev>0.0003923</bias_stddev>
@@ -96,18 +96,18 @@
                     </x>
                     <y>
-                    <noise type="gaussian">
-                        <mean>0.0</mean>
-                        <stddev>0.0001373</stddev>
-                        <bias_mean>0.0</bias_mean>
-                        <bias_stddev>0.0003923</bias_stddev>
-                    </noise>
-                    </y>
-                    <z>
-                    <noise type="gaussian">
-                        <mean>0.0</mean>
-                        <stddev>0.0001373</stddev>
-                        <bias_mean>0.0</bias_mean>
-                        <bias_stddev>0.0003923</bias_stddev>
-                    </noise>
+                        <noise type="gaussian">
+                            <mean>0.0</mean>
+                            <stddev>0.01373</stddev>
+                            <bias_mean>0.0</bias_mean>
+                            <bias_stddev>0.0003923</bias_stddev>
+                        </noise>
+                    </y>
+                    <z>
+                        <noise type="gaussian">
+                            <mean>0.0</mean>
+                            <stddev>0.01373</stddev>
+                            <bias_mean>0.0</bias_mean>
+                            <bias_stddev>0.0003923</bias_stddev>
+                        </noise>
                     </z>
                 </linear_acceleration>
@@ -139,5 +139,5 @@
                             <stddev>0.001745329251</stddev>
                             <bias_mean>0.0</bias_mean>
-                            <bias_stddev>0.01745329251</bias_stddev>
+                            <bias_stddev>0.01745329251</bias_stddev> <!-- 0.01745329251-->
                         </noise>
                     </y>
@@ -155,21 +155,21 @@
                         <noise type="gaussian">
                             <mean>0.0</mean>    <!-- 100 ODR(Output Data Rate) için 32hz bandwith-->
-                            <stddev>0.0014715</stddev> <!-- Output Noise Density, m/s^2 cinsinde, sensorün tipik davranışı ele alınmıştır. -->
-                            <bias_mean>0.0</bias_mean>
-                            <bias_stddev>0.785</bias_stddev> <!-- zero g offset: Burada, imu hareket etmediği halde üretilen gürültüdür. -->
-                        </noise>
-                    </x>
-                    <y>
-                    <noise type="gaussian">
-                        <mean>0.0</mean>
-                        <stddev>0.0014715</stddev>
-                        <bias_mean>0.0</bias_mean>
-                        <bias_stddev>0.785</bias_stddev>
-                    </noise>
-                    </y>
-                    <z>
-                    <noise type="gaussian">
-                        <mean>0.0</mean>
-                        <stddev>0.0014715</stddev>
+                            <stddev>0.0015</stddev> <!-- Output Noise Density, m/s^2 cinsinde, sensorün tipik davranışı ele alınmıştır. -->
+                            <bias_mean>0.0</bias_mean>
+                            <bias_stddev>0.7848</bias_stddev> <!-- zero g offset: Burada, imu hareket etmediği halde üretilen gürültüdür. -->
+                        </noise>
+                    </x>
+                    <y>
+                    <noise type="gaussian">
+                        <mean>0.0</mean>
+                        <stddev>0.0015</stddev>
+                        <bias_mean>0.0</bias_mean>
+                        <bias_stddev>0.7848</bias_stddev>
+                    </noise>
+                    </y>
+                    <z>
+                    <noise type="gaussian">
+                        <mean>0.0</mean>
+                        <stddev>0.0015</stddev>
                         <bias_mean>0.0</bias_mean>
                         <bias_stddev>0.7848</bias_stddev>
@@ -217,23 +217,23 @@
                         <noise type="gaussian">
                             <mean>0.0</mean>    <!-- 100 ODR(Output Data Rate) için 32hz bandwith-->
-                            <stddev>0.0014715</stddev> <!-- Output Noise Density, m/s^2 cinsinde, sensorün tipik davranışı ele alınmıştır. -->
-                            <bias_mean>0.0</bias_mean>
-                            <bias_stddev>0.4903</bias_stddev>
-                        </noise>
-                    </x>
-                    <y>
-                    <noise type="gaussian">
-                        <mean>0.0</mean>
-                        <stddev>0.0014715</stddev>
-                        <bias_mean>0.0</bias_mean>
-                        <bias_stddev>1.471e-3</bias_stddev>
-                    </noise>
-                    </y>
-                    <z>
-                    <noise type="gaussian">
-                        <mean>0.0</mean>
-                        <stddev>0.0014715</stddev>
-                        <bias_mean>0.0</bias_mean>
-                        <bias_stddev>1.471e-3</bias_stddev>
+                            <stddev>0.0015</stddev> <!-- Output Noise Density, m/s^2 cinsinde, sensorün tipik davranışı ele alınmıştır. -->
+                            <bias_mean>0.0</bias_mean>
+                            <bias_stddev>0.7848</bias_stddev> <!-- zero g offset: Burada, imu hareket etmediği halde üretilen gürültüdür. -->
+                        </noise>
+                    </x>
+                    <y>
+                    <noise type="gaussian">
+                        <mean>0.0</mean>
+                        <stddev>0.0015</stddev>
+                        <bias_mean>0.0</bias_mean>
+                        <bias_stddev>0.7848</bias_stddev>
+                    </noise>
+                    </y>
+                    <z>
+                    <noise type="gaussian">
+                        <mean>0.0</mean>
+                        <stddev>0.0015</stddev>
+                        <bias_mean>0.0</bias_mean>
+                        <bias_stddev>0.7848</bias_stddev>
                     </noise>
                     </z>

Commit message: Tüm hatalar düzeltilmiş olup, test ortamı hazırlanmış ve testler düzgün şekilde gerçekleştirilmiştir

File: pilbot_description/urdf/pilbot.urdf.xacro (robot description, xacro)
@@ -195,5 +195,5 @@
     </link>
     <joint name="imu_joint2" type="fixed">
-        <origin xyz="0 0 0.07" rpy="0 0 0"/>
+        <origin xyz="0 0 0.07003" rpy="0 0 0"/>
         <parent link="base_link"/>
         <child link="imu_link2"/>
@@ -222,5 +222,5 @@
     </link>
     <joint name="imu_joint3" type="fixed">
-        <origin xyz="0 0 0.07" rpy="0 0 0"/>
+        <origin xyz="0 0 0.07006" rpy="0 0 0"/>
         <parent link="base_link"/>
         <child link="imu_link3"/>

File: pilbot_description/urdf/pilbot_gazebo.xacro (robot description, xacro)
@@ -64,5 +64,5 @@
                         <noise type="gaussian">
                             <mean>0.0</mean>
-                            <stddev>0.0006109</stddev>
+                            <stddev>0.000006109</stddev>
                             <bias_mean>0.0</bias_mean>
                             <bias_stddev>0.00004848</bias_stddev>
@@ -72,5 +72,5 @@
                         <noise type="gaussian">
                             <mean>0.0</mean>
-                            <stddev>0.0006109</stddev>
+                            <stddev>0.000006109</stddev>
                             <bias_mean>0.0</bias_mean>
                             <bias_stddev>0.00004848</bias_stddev>
@@ -80,5 +80,5 @@
                         <noise type="gaussian">
                             <mean>0.0</mean>
-                            <stddev>0.0006109</stddev>
+                            <stddev>0.000006109</stddev>
                             <bias_mean>0.0</bias_mean>
                             <bias_stddev>0.00004848</bias_stddev>
@@ -90,23 +90,23 @@
                         <noise type="gaussian">
                             <mean>0.0</mean>
-                            <stddev>0.01373</stddev>
-                            <bias_mean>0.0</bias_mean>
-                            <bias_stddev>0.0003923</bias_stddev>
-                        </noise>
-                    </x>
-                    <y>
-                        <noise type="gaussian">
-                            <mean>0.0</mean>
-                            <stddev>0.01373</stddev>
-                            <bias_mean>0.0</bias_mean>
-                            <bias_stddev>0.0003923</bias_stddev>
-                        </noise>
-                    </y>
-                    <z>
-                        <noise type="gaussian">
-                            <mean>0.0</mean>
-                            <stddev>0.01373</stddev>
-                            <bias_mean>0.0</bias_mean>
-                            <bias_stddev>0.0003923</bias_stddev>
+                            <stddev>0.0013734</stddev>
+                            <bias_mean>0.0</bias_mean>
+                            <bias_stddev>0.0004</bias_stddev> <!-- 0.0003923-->
+                        </noise>
+                    </x>
+                    <y>
+                        <noise type="gaussian">
+                            <mean>0.0</mean>
+                            <stddev>0.0013734</stddev>
+                            <bias_mean>0.0</bias_mean>
+                            <bias_stddev>0.0004</bias_stddev>
+                        </noise>
+                    </y>
+                    <z>
+                        <noise type="gaussian">
+                            <mean>0.0</mean>
+                            <stddev>0.0013734</stddev>
+                            <bias_mean>0.0</bias_mean>
+                            <bias_stddev>0.0004</bias_stddev>
                         </noise>
                     </z>
@@ -131,21 +131,21 @@
                             <stddev>0.001745329251</stddev>  <!-- Noise Density, radyan cinsinden! (sensörün tipik davranışı modellenmiştir) -->
                             <bias_mean>0.0</bias_mean>
-                            <bias_stddev>0.01745329251</bias_stddev> <!-- Bias instability, radyan cinsinden! (sensörün tipik davranışı modellenmiştir) -->
-                        </noise>
-                    </x>
-                    <y>
-                        <noise type="gaussian">
-                            <mean>0.0</mean>
-                            <stddev>0.001745329251</stddev>
-                            <bias_mean>0.0</bias_mean>
-                            <bias_stddev>0.01745329251</bias_stddev> <!-- 0.01745329251-->
-                        </noise>
-                    </y>
-                    <z>
-                        <noise type="gaussian">
-                            <mean>0.0</mean>
-                            <stddev>0.001745329251</stddev>
-                            <bias_mean>0.0</bias_mean>
-                            <bias_stddev>0.01745329251</bias_stddev>
+                            <bias_stddev>0.0035</bias_stddev> <!-- Bias instability, radyan cinsinden! (sensörün tipik davranışı modellenmiştir) -->
+                        </noise>
+                    </x>
+                    <y>
+                        <noise type="gaussian">
+                            <mean>0.0</mean>
+                            <stddev>0.001745329251</stddev>
+                            <bias_mean>0.0</bias_mean>
+                            <bias_stddev>0.0035</bias_stddev> <!-- 0.01745329251-->
+                        </noise>
+                    </y>
+                    <z>
+                        <noise type="gaussian">
+                            <mean>0.0</mean>
+                            <stddev>0.001745329251</stddev>
+                            <bias_mean>0.0</bias_mean>
+                            <bias_stddev>0.0035</bias_stddev> <!-- 10 üssü -5 -->
                         </noise>
                     </z>
@@ -157,22 +157,22 @@
                             <stddev>0.0015</stddev> <!-- Output Noise Density, m/s^2 cinsinde, sensorün tipik davranışı ele alınmıştır. -->
                             <bias_mean>0.0</bias_mean>
-                            <bias_stddev>0.7848</bias_stddev> <!-- zero g offset: Burada, imu hareket etmediği halde üretilen gürültüdür. -->
-                        </noise>
-                    </x>
-                    <y>
-                    <noise type="gaussian">
-                        <mean>0.0</mean>
-                        <stddev>0.0015</stddev>
-                        <bias_mean>0.0</bias_mean>
-                        <bias_stddev>0.7848</bias_stddev>
-                    </noise>
-                    </y>
-                    <z>
-                    <noise type="gaussian">
-                        <mean>0.0</mean>
-                        <stddev>0.0015</stddev>
-                        <bias_mean>0.0</bias_mean>
-                        <bias_stddev>0.7848</bias_stddev>
-                    </noise>
+                            <bias_stddev>0.008</bias_stddev>  <!-- zero g offset: Burada, imu hareket etmediği halde üretilen gürültüdür. -->
+                        </noise>
+                    </x>
+                    <y>
+                        <noise type="gaussian">
+                            <mean>0.0</mean>
+                            <stddev>0.0015</stddev>
+                            <bias_mean>0.0</bias_mean>
+                            <bias_stddev>0.008</bias_stddev>
+                        </noise>
+                    </y>
+                    <z>
+                        <noise type="gaussian">
+                            <mean>0.0</mean>
+                            <stddev>0.0015</stddev>
+                            <bias_mean>0.0</bias_mean>
+                            <bias_stddev>0.008</bias_stddev>
+                        </noise>
                     </z>
                 </linear_acceleration>
@@ -193,21 +193,21 @@
                             <stddev>0.001745329251</stddev>  <!-- Noise Density, radyan cinsinden! (sensörün tipik davranışı modellenmiştir) -->
                             <bias_mean>0.0</bias_mean>
-                            <bias_stddev>0.01745329251</bias_stddev> <!-- Bias instability, radyan cinsinden! (sensörün tipik davranışı modellenmiştir) -->
-                        </noise>
-                    </x>
-                    <y>
-                        <noise type="gaussian">
-                            <mean>0.0</mean>
-                            <stddev>0.001745329251</stddev>
-                            <bias_mean>0.0</bias_mean>
-                            <bias_stddev>0.01745329251</bias_stddev>
-                        </noise>
-                    </y>
-                    <z>
-                        <noise type="gaussian">
-                            <mean>0.0</mean>
-                            <stddev>0.001745329251</stddev>
-                            <bias_mean>0.0</bias_mean>
-                            <bias_stddev>0.01745329251</bias_stddev>
+                            <bias_stddev>0.0035</bias_stddev> <!-- Bias instability, radyan cinsinden! (sensörün tipik davranışı modellenmiştir) -->
+                        </noise>
+                    </x>
+                    <y>
+                        <noise type="gaussian">
+                            <mean>0.0</mean>
+                            <stddev>0.001745329251</stddev>
+                            <bias_mean>0.0</bias_mean>
+                            <bias_stddev>0.0035</bias_stddev> <!-- 0.01745329251-->
+                        </noise>
+                    </y>
+                    <z>
+                        <noise type="gaussian">
+                            <mean>0.0</mean>
+                            <stddev>0.001745329251</stddev>
+                            <bias_mean>0.0</bias_mean>
+                            <bias_stddev>0.0035</bias_stddev> <!-- 10 üssü -5 -->
                         </noise>
                     </z>
@@ -219,22 +219,22 @@
                             <stddev>0.0015</stddev> <!-- Output Noise Density, m/s^2 cinsinde, sensorün tipik davranışı ele alınmıştır. -->
                             <bias_mean>0.0</bias_mean>
-                            <bias_stddev>0.7848</bias_stddev> <!-- zero g offset: Burada, imu hareket etmediği halde üretilen gürültüdür. -->
-                        </noise>
-                    </x>
-                    <y>
-                    <noise type="gaussian">
-                        <mean>0.0</mean>
-                        <stddev>0.0015</stddev>
-                        <bias_mean>0.0</bias_mean>
-                        <bias_stddev>0.7848</bias_stddev>
-                    </noise>
-                    </y>
-                    <z>
-                    <noise type="gaussian">
-                        <mean>0.0</mean>
-                        <stddev>0.0015</stddev>
-                        <bias_mean>0.0</bias_mean>
-                        <bias_stddev>0.7848</bias_stddev>
-                    </noise>
+                            <bias_stddev>0.008</bias_stddev> <!-- zero g offset: Burada, imu hareket etmediği halde üretilen gürültüdür. -->
+                        </noise>
+                    </x>
+                    <y>
+                        <noise type="gaussian">
+                            <mean>0.0</mean>
+                            <stddev>0.0015</stddev>
+                            <bias_mean>0.0</bias_mean>
+                            <bias_stddev>0.008</bias_stddev>
+                        </noise>
+                    </y>
+                    <z>
+                        <noise type="gaussian">
+                            <mean>0.0</mean>
+                            <stddev>0.0015</stddev>
+                            <bias_mean>0.0</bias_mean>
+                            <bias_stddev>0.008</bias_stddev>
+                        </noise>
                     </z>
                 </linear_acceleration>
